Commit message: Added laser and multi hero launch

File: hero_description/urdf/hero.xacro (robot description, xacro)
@@ -1,9 +1,10 @@
 <!--?xml version="1.0"?-->
 <robot>
+  <!-- Some properties of HERO -->
   <property name="PI" value="3.1415926535897931" />
   <property name="wheel_separation" value="0.0623" />
   <property name="wheel_radius" value="0.0496" />
-  <property name="height" value="0.085" />
-    <link name="base_link" >
+  <!-- Here was the base link definitions -->
+  <link name="base_link" >
     <visual>
       <origin xyz="0 0 0" rpy="0 0 ${PI}" />
@@ -19,6 +20,6 @@
     </collision>
     <inertial>
-      <mass value="0.087" />
-      <origin xyz="0 0 0" rpy="0 0 0"/>
+      <mass value="0.090" />
+      <origin xyz="0 0 -0.01" rpy="0 0 0"/>
       <inertia ixx="0.00003312" ixy="0" ixz="0"
 	           iyy="0.00003732" iyz="0"
@@ -26,5 +27,10 @@
     </inertial>
   </link>
-  <!--  here was the hat joint and link -->
+  <!--  Here was the hat joint and link -->
+  <joint name="hat_joint" type="fixed">
+      <origin xyz="0.0001 0 0.038" rpy="0 0 0" />
+      <parent link="base_link"/>
+      <child link="hat_link"/>
+  </joint>
   <link name="hat_link" >
     <visual>
@@ -48,14 +54,9 @@
          </inertial>
   </link>
-  <!--  here was the left wheel joint and link -->
-  <joint name="hat_joint" type="fixed">
-      <origin xyz="0.0001 0 0.038" rpy="0 0 0" />
-      <parent link="base_link"/>
-      <child link="hat_link"/>
-  </joint>
+  <!--  Here was the left wheel joint and link -->
   <joint name="left_wheel_joint" type="continuous">
       <parent link="base_link"/>
       <child link="left_wheel_link"/>
-      <origin xyz="0 ${-wheel_separation/2} 0" rpy="0 0 0" />
+      <origin xyz="0 ${-wheel_separation/2} 0.0005" rpy="0 0 0" />
       <axis xyz="0 1 0" />
       <limit effort="1" velocity="0.3"/>
@@ -84,10 +85,10 @@
     </inertial>
   </link>
-  <!--  here was the right wheel joint and link -->
+  <!--  Here was the right wheel joint and link -->
   <joint name="right_wheel_joint" type="continuous">
       <axis xyz="0 1 0" />
       <limit effort="1" velocity="0.3"/>
       <dynamics damping="0.0" friction="0" />
-      <origin xyz="0 ${wheel_separation/2} 0" rpy="0 0 0" />
+      <origin xyz="0 ${wheel_separation/2} 0.0005" rpy="0 0 0" />
       <parent link="base_link"/>
       <child link="right_wheel_link"/>
@@ -114,16 +115,16 @@
       </inertial>
   </link>
-  <!--joint name="board_joint" type="fixed">
+  <joint name="laser_joint" type="fixed">
     <axis xyz="0 1 0" />
-    <origin xyz="0 0 ${height3 - axel_offset/2}" rpy="0 0 0"/>
-    <parent link="link3"/>
-    <child link="hokuyo_link"/>
-  </joint-->
-  <!-- Hokuyo Laser -->
-  <!--link name="board_link">
+    <origin xyz="0 0 0.031" rpy="0 0 0"/>
+    <parent link="base_link"/>
+    <child link="laser_link"/>
+  </joint>
+  <!-- Here is the laser link -->
+  <link name="laser_link">
     <collision>
       <origin xyz="0 0 0" rpy="0 0 0"/>
       <geometry>
-        <box size="0.1 0.1 0.1"/>
+        <box size="0.001 0.001 0.001"/>
       </geometry>
     </collision>
@@ -131,5 +132,5 @@
       <origin xyz="0 0 0" rpy="0 0 0"/>
       <geometry>
-        <box size="0.1 0.1 0.1"/>
+        <box size="0.001 0.001 0.001"/>
       </geometry>
     </visual>
@@ -139,5 +140,6 @@
       <inertia ixx="1e-6" ixy="0" ixz="0" iyy="1e-6" iyz="0" izz="1e-6" />
     </inertial>
-  </link-->
+  </link>
+ <!-- Here is the left joint transmission to gazebo -->
  <transmission name="left_wheel_tran">
     <type>transmission_interface/SimpleTransmission</type>
@@ -147,8 +149,9 @@
     <actuator name="left_wheel_motor">
       <mechanicalReduction>1</mechanicalReduction>
-      <!--hardwareInterface>VelocityJointInterface</hardwareInterface-->
+      <hardwareInterface>hardware_interface/EffortJointInterface</hardwareInterface>
     </actuator>
-  </transmission>
-  <transmission name="right_wheel_tran">
+ </transmission>
+ <!-- Here is the right joint transmission to gazebo -->
+ <transmission name="right_wheel_tran">
     <type>transmission_interface/SimpleTransmission</type>
     <joint name="right_wheel_joint">
@@ -157,5 +160,5 @@
     <actuator name="right_wheel_motor">
       <mechanicalReduction>1</mechanicalReduction>
-      <!--hardwareInterface>VelocityJointInterface</hardwareInterface-->
+      <hardwareInterface>hardware_interface/EffortJointInterface</hardwareInterface>
     </actuator>
   </transmission>
