Commit message: Improve gazebo simulation setup; add swarm arena setup;

File: hero_description/urdf/common.xacro (robot description, xacro)
@@ -4,5 +4,6 @@
   <property name="PI" value="3.1415926535897931" />
   <property name="wheel_separation" value="0.0623" />
-  <property name="wheel_diameter" value="0.0496" />
+  <!-- <property name="wheel_diameter" value="0.0496" /> -->
+  <property name="wheel_diameter" value="0.052" />
   <macro name="cylinder_inertia" params="m r h">
     <inertia ixx="${m*(3*r*r+h*h)/12}" ixy = "0" ixz = "0" iyy="${m*(3*r*r+h*h)/12}" iyz = "0" izz="${m*r*r/2}" />

File: hero_description/urdf/hero.gazebo.xacro (robot description, xacro)
@@ -13,5 +13,5 @@
       <!--robotNamespace>/</robotNamespace-->
       <alwaysOn>true</alwaysOn>
-      <updateRate>100</updateRate>
+      <updateRate>50</updateRate>
       <leftJoint>left_wheel_joint</leftJoint>
       <rightJoint>right_wheel_joint</rightJoint>
@@ -29,7 +29,7 @@
       <publishWheelTF>true</publishWheelTF>
       <publishWheelJointState>false</publishWheelJointState>
-      <wheelAcceleration>0</wheelAcceleration>
+      <wheelAcceleration>0.0</wheelAcceleration>
       <publishTf>true</publishTf>
-      <wheelTorque>0.3</wheelTorque>
+      <wheelTorque>2.5</wheelTorque>
     </plugin>
   </gazebo>
@@ -40,5 +40,5 @@
         <!--robotNamespace>/</robotNamespace-->
         <serviceName>hat_color</serviceName>
-        <color>1.0 1.0 1.0 1.0</color>
+        <color>0.0 0.5 0.9 1.0</color>
       </plugin>
     </visual>

File: hero_description/urdf/hero.xacro (robot description, xacro)
@@ -12,5 +12,6 @@
       <origin xyz="0 0 0" rpy="0 0 ${PI}" />
       <geometry>
-        <box size="0.068 0.068 0.048"/>
+        <!-- <cylinde size="0.068 0.068 0.048"/> -->
+        <cylinder length="0.048" radius="0.036"/>
       </geometry>
     </collision>
@@ -18,7 +19,13 @@
       <mass value="0.090" />
       <origin xyz="0 0 0" rpy="0 0 0"/>
-      <xacro:box_inertia m="0.090" x="0.068" y="0.068" z="0.055"/>
+      <xacro:cylinder_inertia m="0.090" r="0.035" h="0.055"/>
     </inertial>
   </link>
+  <gazebo reference="base_link">
+    <gravity>1</gravity>
+    <mu1 value="0.01"/>
+    <mu2 value="0.01"/>
+    <!-- <maxVel value="0.10"/>  -->
+  </gazebo>
   <!--  Here was the hat joint and link -->
   <joint name="hat_joint" type="fixed">
@@ -37,5 +44,6 @@
       <origin xyz="0 0 0" rpy="0 0 0" />
       <geometry>
-        <box size="0.068 0.068 0.02"/>
+        <!-- <box size="0.068 0.068 0.02"/> -->
+        <cylinder length="0.02" radius="0.040"/>
       </geometry>
     </collision>
@@ -43,17 +51,61 @@
       <mass value="0.010" />
       <origin xyz="0 0 0" rpy="0 0 0"/>
-      <xacro:box_inertia m="0.010" x="0.07" y="0.07" z="0.02"/>
+      <!-- <xacro:box_inertia m="0.010" x="0.07" y="0.07" z="0.02"/> -->
+      <xacro:cylinder_inertia m="0.010" r="0.035" h="0.02"/>
     </inertial>
   </link>
+  <gazebo reference="hat_link">
+    <gravity>1</gravity>
+    <!-- <mu1 value="0.005"/>
+    <mu2 value="0.005"/> -->
+    <maxVel value="0.10"/>
+  </gazebo>
   <!--  Here was the left wheel joint and link -->
   <joint name="left_wheel_joint" type="continuous">
     <parent link="base_link"/>
     <child link="left_wheel_link"/>
-    <origin xyz="0 ${-wheel_separation/2} 0.0005" rpy="0 0 0" />
+    <origin xyz="0 ${wheel_separation/2} 0.0005" rpy="0 0 0" />
     <axis xyz="0 1 0" />
-    <limit effort="1" velocity="0.3"/>
+    <limit effort="100" velocity="0.3"/>
     <dynamics damping="0.0" friction="0.0" />
   </joint>
   <link name="left_wheel_link">
+    <visual>
+      <origin xyz="0 0 0.0" rpy="${PI/2} 0 0" />
+      <geometry>
+        <mesh filename="package://hero_description/meshes/wheel.dae" scale="1 1 1"/>
+      </geometry>
+    </visual>
+    <collision>
+      <origin xyz="0 0 0.0" rpy="${PI/2} 0 0" />
+      <geometry>
+        <cylinder length="0.008" radius="${wheel_diameter/2.0}"/>
+      </geometry>
+    </collision>
+    <inertial>
+      <mass value="0.010" />
+      <origin xyz="0 0 0" rpy="${PI/2} 0 0"/>
+      <xacro:cylinder_inertia m="0.010" h="0.008" r="${wheel_diameter/2.0}"/>
+    </inertial>
+  </link>
+  <gazebo reference="left_wheel_link">
+    <mu1 value="0.8"/>
+    <mu2 value="0.8"/>
+    <!-- <maxVel value="0.10"/>  -->
+    <!-- <kp value="10000000.0"/>
+    <kd value="1.0"/>
+    <fdir1 value="1 0 0"/> -->
+    <gravity>1</gravity>
+  </gazebo>
+  <!--  Here was the right wheel joint and link -->
+  <joint name="right_wheel_joint" type="continuous">
+    <axis xyz="0 1 0" />
+    <limit effort="100" velocity="0.3"/>
+    <dynamics damping="0.0" friction="0" />
+    <origin xyz="0 ${-wheel_separation/2} 0.0005" rpy="0 0 0" />
+    <parent link="base_link"/>
+    <child link="right_wheel_link"/>
+  </joint>
+  <link name="right_wheel_link">
     <visual>
       <origin xyz="0 0 0.0" rpy="${-PI/2} 0 0" />
@@ -74,31 +126,12 @@
     </inertial>
   </link>
-  <!--  Here was the right wheel joint and link -->
-  <joint name="right_wheel_joint" type="continuous">
-    <axis xyz="0 1 0" />
-    <limit effort="1" velocity="0.3"/>
-    <dynamics damping="0.0" friction="0" />
-    <origin xyz="0 ${wheel_separation/2} 0.0005" rpy="0 0 0" />
-    <parent link="base_link"/>
-    <child link="right_wheel_link"/>
-  </joint>
-  <link name="right_wheel_link">
-    <visual>
-      <origin xyz="0 0 0.0" rpy="${PI/2} 0 0" />
-      <geometry>
-        <mesh filename="package://hero_description/meshes/wheel.dae" scale="1 1 1"/>
-      </geometry>
-    </visual>
-    <collision>
-      <origin xyz="0 0 0.0" rpy="${PI/2} 0 0" />
-      <geometry>
-        <cylinder length="0.008" radius="${wheel_diameter/2.0}"/>
-      </geometry>
-    </collision>
-    <inertial>
-      <mass value="0.010" />
-      <origin xyz="0 0 0" rpy="${PI/2} 0 0"/>
-      <xacro:cylinder_inertia m="0.010" h="0.008" r="${wheel_diameter/2.0}"/>
-    </inertial>
-  </link>
+  <gazebo reference="right_wheel_link">
+    <mu1 value="0.8"/>
+    <mu2 value="0.8"/>
+    <!-- <maxVel value="0.10"/>  -->
+    <!-- <kp value="10000000.0"/>
+    <kd value="1.0"/>
+    <fdir1 value="1 0 0"/> -->
+    <gravity>1</gravity>
+  </gazebo>
 </robot>

File: hero_description/urdf/laser.gazebo.xacro (robot description, xacro)
@@ -6,5 +6,5 @@
             <pose>0 0 0.031 0 0 0</pose>
             <visualize>true</visualize>
-            <update_rate>40</update_rate>
+            <update_rate>10</update_rate>
             <ray>
                 <scan>
@@ -26,5 +26,5 @@
                 <frameName>laser_link</frameName>
                 <gaussianNoise>0.001</gaussianNoise>
-                <updateRate>30</updateRate>
+                <updateRate>20</updateRate>
             </plugin>
         </sensor>

Commit message: Major Modifications

File: hero_description/urdf/common.xacro (robot description, xacro)
@@ -3,7 +3,7 @@
   <!-- Some properties of HERO -->
   <property name="PI" value="3.1415926535897931" />
-  <property name="wheel_separation" value="0.0623" />
+  <property name="wheel_separation" value="0.06460" />
   <!-- <property name="wheel_diameter" value="0.0496" /> -->
-  <property name="wheel_diameter" value="0.052" />
+  <property name="wheel_diameter" value="0.050" />
   <macro name="cylinder_inertia" params="m r h">
     <inertia ixx="${m*(3*r*r+h*h)/12}" ixy = "0" ixz = "0" iyy="${m*(3*r*r+h*h)/12}" iyz = "0" izz="${m*r*r/2}" />

File: hero_description/urdf/hero.gazebo.xacro (robot description, xacro)
@@ -6,4 +6,5 @@
       <!--robotNamespace>/</robotNamespace-->
       <legacyModeNS>true</legacyModeNS>
+      <controlPeriod>0.60</controlPeriod>
     </plugin>
   </gazebo>
@@ -13,10 +14,10 @@
       <!--robotNamespace>/</robotNamespace-->
       <alwaysOn>true</alwaysOn>
-      <updateRate>50</updateRate>
+      <updateRate>15</updateRate>
       <leftJoint>left_wheel_joint</leftJoint>
       <rightJoint>right_wheel_joint</rightJoint>
       <wheelSeparation>${wheel_separation}</wheelSeparation>
       <wheelDiameter>${wheel_diameter}</wheelDiameter>
-      <torque>0.3</torque>
+      <torque>0.03</torque>
       <commandTopic>cmd_vel</commandTopic>
       <odometryTopic>odom</odometryTopic>
@@ -31,5 +32,5 @@
       <wheelAcceleration>0.0</wheelAcceleration>
       <publishTf>true</publishTf>
-      <wheelTorque>2.5</wheelTorque>
+      <wheelTorque>0.5</wheelTorque>
     </plugin>
   </gazebo>
@@ -37,7 +38,8 @@
   <gazebo reference='hat_link'>
     <visual>
-      <plugin name="gazebo_ros_model_color" filename="libgazebo_ros_model_color.so">
+      <plugin name="libgazebo_ros_hero_color" filename="libgazebo_ros_hero_color.so">
         <!--robotNamespace>/</robotNamespace-->
         <serviceName>hat_color</serviceName>
+        <topicName>hat_color</topicName>
         <color>0.0 0.5 0.9 1.0</color>
       </plugin>

File: hero_description/urdf/hero.xacro (robot description, xacro)
@@ -4,20 +4,21 @@
   <link name="base_link">
     <visual>
-      <origin xyz="0 0 0" rpy="0 0 ${PI}" />
+      <origin xyz="0 0 0" rpy="0 0 ${pi/2}" />
       <geometry>
-        <mesh filename="package://hero_description/meshes/base_link.dae" scale="1 1 1"/>
+        <mesh filename="package://hero_description/meshes/base_link.obj" scale="1 1 1"/>
       </geometry>
     </visual>
     <collision>
-      <origin xyz="0 0 0" rpy="0 0 ${PI}" />
+      <origin xyz="0 0 0.0121" rpy="0 0 ${pi/2}" />
       <geometry>
         <!-- <cylinde size="0.068 0.068 0.048"/> -->
-        <cylinder length="0.048" radius="0.036"/>
+        <cylinder length="0.042" radius="0.037"/>
+        <!-- <mesh filename="package://hero_description/meshes/base_link.dae" scale="1 1 1"/> -->
       </geometry>
     </collision>
     <inertial>
       <mass value="0.090" />
-      <origin xyz="0 0 0" rpy="0 0 0"/>
-      <xacro:cylinder_inertia m="0.090" r="0.035" h="0.055"/>
+      <origin xyz="0 0.0002 0" rpy="${pi/2} 0 0"/>
+      <xacro:cylinder_inertia m="0.090" r="0.035" h="0.065"/>
     </inertial>
   </link>
@@ -27,8 +28,10 @@
     <mu2 value="0.01"/>
     <!-- <maxVel value="0.10"/>  -->
+    <maxContacts>4</maxContacts>
+    <selfCollide>1</selfCollide>
   </gazebo>
   <!--  Here was the hat joint and link -->
   <joint name="hat_joint" type="fixed">
-    <origin xyz="0.0001 0 0.038" rpy="0 0 0" />
+    <origin xyz="-0.00245 -0.00216 0.06027" rpy="0 0 0" />
     <parent link="base_link"/>
     <child link="hat_link"/>
@@ -38,5 +41,5 @@
       <origin xyz="0 0 0" rpy="0 0 0" />
       <geometry>
-        <mesh filename="package://hero_description/meshes/hat.dae" scale="1 1 1"/>
+        <mesh filename="package://hero_description/meshes/hat.obj" scale="1 1 1"/>
       </geometry>
     </visual>
@@ -45,5 +48,6 @@
       <geometry>
         <!-- <box size="0.068 0.068 0.02"/> -->
-        <cylinder length="0.02" radius="0.040"/>
+        <!-- <cylinder length="0.02" radius="0.040"/> -->
+        <mesh filename="package://hero_description/meshes/hat.obj" scale="1 1 1"/>
       </geometry>
     </collision>
@@ -60,4 +64,6 @@
     <mu2 value="0.005"/> -->
     <maxVel value="0.10"/>
+    <maxContacts>0</maxContacts>
+    <selfCollide>0</selfCollide>
   </gazebo>
   <!--  Here was the left wheel joint and link -->
@@ -65,14 +71,14 @@
     <parent link="base_link"/>
     <child link="left_wheel_link"/>
-    <origin xyz="0 ${wheel_separation/2} 0.0005" rpy="0 0 0" />
+    <origin xyz="0.0 ${wheel_separation/2} 0.01548" rpy="0 0 0" />
     <axis xyz="0 1 0" />
-    <limit effort="100" velocity="0.3"/>
-    <dynamics damping="0.0" friction="0.0" />
+    <limit effort="0.1" velocity="0.3"/>
+    <dynamics damping="0.0001" friction="0.0" />
   </joint>
   <link name="left_wheel_link">
     <visual>
-      <origin xyz="0 0 0.0" rpy="${PI/2} 0 0" />
+      <origin xyz="0 0 0.0" rpy="0 0 0" />
       <geometry>
-        <mesh filename="package://hero_description/meshes/wheel.dae" scale="1 1 1"/>
+        <mesh filename="package://hero_description/meshes/wheel.obj" scale="1 1 1"/>
       </geometry>
     </visual>
@@ -84,5 +90,5 @@
     </collision>
     <inertial>
-      <mass value="0.010" />
+      <mass value="0.020" />
       <origin xyz="0 0 0" rpy="${PI/2} 0 0"/>
       <xacro:cylinder_inertia m="0.010" h="0.008" r="${wheel_diameter/2.0}"/>
@@ -90,6 +96,6 @@
   </link>
   <gazebo reference="left_wheel_link">
-    <mu1 value="0.8"/>
-    <mu2 value="0.8"/>
+    <mu1 value="1.0"/>
+    <mu2 value="1.0"/>
     <!-- <maxVel value="0.10"/>  -->
     <!-- <kp value="10000000.0"/>
@@ -97,11 +103,13 @@
     <fdir1 value="1 0 0"/> -->
     <gravity>1</gravity>
+    <maxContacts>4</maxContacts>
+    <selfCollide>0</selfCollide>
   </gazebo>
   <!--  Here was the right wheel joint and link -->
   <joint name="right_wheel_joint" type="continuous">
     <axis xyz="0 1 0" />
-    <limit effort="100" velocity="0.3"/>
-    <dynamics damping="0.0" friction="0" />
-    <origin xyz="0 ${-wheel_separation/2} 0.0005" rpy="0 0 0" />
+    <limit effort="0.1" velocity="0.3"/>
+    <dynamics damping="0.0001" friction="0" />
+    <origin xyz="0.0 ${-wheel_separation/2} 0.01548" rpy="0 0 0" />
     <parent link="base_link"/>
     <child link="right_wheel_link"/>
@@ -109,7 +117,7 @@
   <link name="right_wheel_link">
     <visual>
-      <origin xyz="0 0 0.0" rpy="${-PI/2} 0 0" />
+      <origin xyz="0 0 0.0" rpy="${-PI} 0 0" />
       <geometry>
-        <mesh filename="package://hero_description/meshes/wheel.dae" scale="1 1 1"/>
+        <mesh filename="package://hero_description/meshes/wheel.obj" scale="1 1 1"/>
       </geometry>
     </visual>
@@ -121,5 +129,5 @@
     </collision>
     <inertial>
-      <mass value="0.010" />
+      <mass value="0.020" />
       <origin xyz="0 0 0" rpy="${-PI/2} 0 0"/>
       <xacro:cylinder_inertia m="0.010" h="0.008" r="${wheel_diameter/2.0}"/>
@@ -127,6 +135,6 @@
   </link>
   <gazebo reference="right_wheel_link">
-    <mu1 value="0.8"/>
-    <mu2 value="0.8"/>
+    <mu1 value="1.0"/>
+    <mu2 value="1.0"/>
     <!-- <maxVel value="0.10"/>  -->
     <!-- <kp value="10000000.0"/>
@@ -134,4 +142,6 @@
     <fdir1 value="1 0 0"/> -->
     <gravity>1</gravity>
+    <maxContacts>4</maxContacts>
+    <selfCollide>0</selfCollide>
   </gazebo>
 </robot>

File: hero_description/urdf/laser.gazebo.xacro (robot description, xacro)
@@ -3,13 +3,13 @@
     <!-- Laser plugin -->
     <gazebo reference="laser_link">
-        <sensor type="gpu_ray" name="head_laser_sensor">
-            <pose>0 0 0.031 0 0 0</pose>
-            <visualize>true</visualize>
-            <update_rate>10</update_rate>
+        <sensor type="gpu_ray" name="hero_laser_sensor">
+            <pose>0 0 0.051 0 0 0</pose>
+            <visualize>false</visualize>
+            <update_rate>20</update_rate>
             <ray>
                 <scan>
                     <horizontal>
-                        <samples>8</samples>
-                        <resolution>1.2</resolution>
+                        <samples>16</samples>
+                        <resolution>1</resolution>
                         <min_angle>${-PI}</min_angle>
                         <max_angle>${PI}</max_angle>
@@ -19,9 +19,9 @@
                     <min>0.038</min>
                     <max>0.20</max>
-                    <resolution>0.01</resolution>
+                    <resolution>0.04</resolution>
                 </range>
             </ray>
-            <plugin name="gazebo_ros_head_hokuyo_controller" filename="libgazebo_ros_gpu_laser.so">
-                <topicName>laser_scan</topicName>
+            <plugin name="gazebo_ros_hero_laser" filename="libgazebo_ros_gpu_laser.so">
+                <topicName>laser</topicName>
                 <frameName>laser_link</frameName>
                 <gaussianNoise>0.001</gaussianNoise>

File: hero_description/urdf/laser.xacro (robot description, xacro)
@@ -3,5 +3,5 @@
     <joint name="laser_joint" type="fixed">
         <axis xyz="0 1 0" />
-        <origin xyz="0 0 0.031" rpy="0 0 0"/>
+        <origin xyz="0 0 0.051" rpy="0 0 0"/>
         <parent link="base_link"/>
         <child link="laser_link"/>

Commit message: Fix xacro urdf remapping #18, thanks @jacobh2299

File: hero_description/urdf/common.xacro (robot description, xacro)
@@ -2,13 +2,13 @@
 <robot xmlns:xacro="http://www.ros.org/wiki/xacro">
   <!-- Some properties of HERO -->
-  <property name="PI" value="3.1415926535897931" />
-  <property name="wheel_separation" value="0.06460" />
+  <xacro:property name="PI" value="3.1415926535897931" />
+  <xacro:property name="wheel_separation" value="0.06460" />
   <!-- <property name="wheel_diameter" value="0.0496" /> -->
-  <property name="wheel_diameter" value="0.050" />
-  <macro name="cylinder_inertia" params="m r h">
+  <xacro:property name="wheel_diameter" value="0.050" />
+  <xacro:macro name="cylinder_inertia" params="m r h">
     <inertia ixx="${m*(3*r*r+h*h)/12}" ixy = "0" ixz = "0" iyy="${m*(3*r*r+h*h)/12}" iyz = "0" izz="${m*r*r/2}" />
-  </macro>
-  <macro name="box_inertia" params="m x y z">
+  </xacro:macro>
+  <xacro:macro name="box_inertia" params="m x y z">
     <inertia ixx="${m*(y*y+z*z)/12}" ixy = "0" ixz = "0" iyy="${m*(x*x+z*z)/12}" iyz = "0" izz="${m*(x*x+z*z)/12}" />
-  </macro>
+  </xacro:macro>
 </robot>

Commit message: Update docker and launch files

File: hero_description/urdf/common.xacro (robot description, xacro)
@@ -2,13 +2,13 @@
 <robot xmlns:xacro="http://www.ros.org/wiki/xacro">
   <!-- Some properties of HERO -->
-  <xacro:property name="PI" value="3.1415926535897931" />
-  <xacro:property name="wheel_separation" value="0.06460" />
+  <property name="PI" value="3.1415926535897931" />
+  <property name="wheel_separation" value="0.06460" />
   <!-- <property name="wheel_diameter" value="0.0496" /> -->
-  <xacro:property name="wheel_diameter" value="0.050" />
-  <xacro:macro name="cylinder_inertia" params="m r h">
+  <property name="wheel_diameter" value="0.050" />
+  <macro name="cylinder_inertia" params="m r h">
     <inertia ixx="${m*(3*r*r+h*h)/12}" ixy = "0" ixz = "0" iyy="${m*(3*r*r+h*h)/12}" iyz = "0" izz="${m*r*r/2}" />
-  </xacro:macro>
-  <xacro:macro name="box_inertia" params="m x y z">
+  </macro>
+  <macro name="box_inertia" params="m x y z">
     <inertia ixx="${m*(y*y+z*z)/12}" ixy = "0" ixz = "0" iyy="${m*(x*x+z*z)/12}" iyz = "0" izz="${m*(x*x+z*z)/12}" />
-  </xacro:macro>
+  </macro>
 </robot>
