File: hero_resources/schematic/EAGLE/projects/hero_v2.6/board.brd (EAGLE design)
At the start: 61.1 x 61.1 mm, 45 parts

Commit message: Update PCB 2.6
Parts:
- moved BATT1 1.06 mm to (35.9, 17.7), flipped to the bottom, turned to 0 degrees
- moved BATT0 0.69 mm to (31.9, 36.2), flipped to the top, turned to 24.7 degrees
- moved R12 0.49 mm to (17.4, 5.06)
- moved STDBY 0.32 mm to (19.6, 5.03)
- moved R13 0.20 mm to (25.0, 5.12)
- moved CHRG 0.15 mm to (22.4, 5.04)
- renumbered I2C|UART to E-HAT
Routing:
- net N$2: track 29.7 -> 27.3 mm, vias 2 -> 1
- net GND: vias 59 -> 61
Other:
- board text added: "TCRT5000"
- board text removed: "2019.04"
- board text removed: "HeRo v2.5"
