File: hero_resources/schematic/EAGLE/projects/hero_v2.6/board.sch (EAGLE design)
At the start: 45 parts

Commit message: Update PCB 2.6
Parts:
- renumbered I2C|UART to E-HAT
Changed lines of the file:
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@@
 <setting verticaltext="up"/>
 </settings>
-<grid distance="0.01" unitdist="inch" unit="inch" style="lines" multiple="1" display="no" altdistance="0.01" altunitdist="inch" altunit="inch"/>
+<grid distance="0.1" unitdist="inch" unit="inch" style="lines" multiple="1" display="no" altdistance="0.01" altunitdist="inch" altunit="inch"/>
 <layers>
 <layer number="1" name="Top" color="4" fill="1" visible="no" active="no"/>
@@
 <part name="GND8" library="supply1" library_urn="urn:adsk.eagle:library:371" deviceset="GND" device=""/>
 <part name="GND9" library="supply1" library_urn="urn:adsk.eagle:library:371" deviceset="GND" device=""/>
-<part name="I2C|UART" library="pinhead" deviceset="PINHD-1X4" device="" package3d_urn="urn:adsk.eagle:package:22407/2"/>
+<part name="E-HAT" library="pinhead" deviceset="PINHD-1X4" device="" package3d_urn="urn:adsk.eagle:package:22407/2"/>
 <part name="GND18" library="supply1" library_urn="urn:adsk.eagle:library:371" deviceset="GND" device=""/>
 <part name="P+22" library="supply1" library_urn="urn:adsk.eagle:library:371" deviceset="VCC" device=""/>
@@
 <attribute name="VALUE" x="-41.91" y="58.42" size="1.778" layer="96" rot="R180"/>
 </instance>
-<instance part="I2C|UART" gate="A" x="71.12" y="69.85" smashed="yes" rot="R180">
+<instance part="E-HAT" gate="A" x="71.12" y="69.85" smashed="yes" rot="R180">
 <attribute name="NAME" x="75.8698" y="61.4172" size="1.778" layer="95" rot="R180"/>
 <attribute name="VALUE" x="77.47" y="77.47" size="1.778" layer="96" rot="R180"/>
@@
 </segment>
 <segment>
-<pinref part="I2C|UART" gate="A" pin="3"/>
+<pinref part="E-HAT" gate="A" pin="3"/>
 <pinref part="GND18" gate="1" pin="GND"/>
 <wire x1="73.66" y1="69.85" x2="93.98" y2="69.85" width="0.1524" layer="91"/>
@@
 </segment>
 <segment>
-<pinref part="I2C|UART" gate="A" pin="4"/>
+<pinref part="E-HAT" gate="A" pin="4"/>
 <wire x1="73.66" y1="72.39" x2="86.36" y2="72.39" width="0.1524" layer="91"/>
 <pinref part="P+22" gate="VCC" pin="VCC"/>
@@
 <net name="SDA_RX" class="0">
 <segment>
-<pinref part="I2C|UART" gate="A" pin="1"/>
+<pinref part="E-HAT" gate="A" pin="1"/>
 <wire x1="73.66" y1="64.77" x2="81.28" y2="64.77" width="0.1524" layer="91"/>
 <label x="81.28" y="64.77" size="0.8128" layer="95" xref="yes"/>
@@
 <net name="SCL_TX" class="0">
 <segment>
-<pinref part="I2C|UART" gate="A" pin="2"/>
+<pinref part="E-HAT" gate="A" pin="2"/>
 <wire x1="73.66" y1="67.31" x2="81.28" y2="67.31" width="0.1524" layer="91"/>
 <label x="81.28" y="67.31" size="0.8128" layer="95" xref="yes"/>
