Commit message: Add new arena environments and maps

File: hero_gazebo/worlds/models/arena_1/arena.urdf (robot description, URDF)
Before this commit: robot arena, 1 links, 0 joints
Links:
- link arena_link: geometry collision mesh filename=package://hero_gazebo/worlds/models/arena_1/arena.obj scale=1 1 1; visual mesh filename=package://hero_gazebo/worlds/models/arena_1/arena.obj scale=1 1 1

File: hero_gazebo/worlds/models/arena_2/arena.urdf (robot description, URDF)
Before this commit: robot arena, 1 links, 0 joints
Links:
- link arena_link: geometry collision mesh filename=package://hero_gazebo/worlds/models/arena_2/arena.obj scale=1 1 1; visual mesh filename=package://hero_gazebo/worlds/models/arena_2/arena.obj scale=1 1 1

File: hero_gazebo/worlds/models/arena_3/arena.urdf (robot description, URDF)
Before this commit: robot arena, 1 links, 0 joints
Links:
- link arena_link: geometry collision mesh filename=package://hero_gazebo/worlds/models/arena_3/arena.obj scale=1 1 1; visual mesh filename=package://hero_gazebo/worlds/models/arena_3/arena.obj scale=1 1 1

File: hero_gazebo/worlds/models/arena_4/arena.urdf (robot description, URDF)
Before this commit: robot arena, 1 links, 0 joints
Links:
- link arena_link: geometry collision mesh filename=package://hero_gazebo/worlds/models/arena_4/arena.obj scale=1 1 1; visual mesh filename=package://hero_gazebo/worlds/models/arena_4/arena.obj scale=1 1 1
