File: hero_resources/schematic/EAGLE/projects/hero_v2.7/board.brd (EAGLE design)
At the start: 61.1 x 61.1 mm, 45 parts

Commit message: Update pcb board version
Parts:
- moved CHRG 48.5 mm to (22.4, 5.04), flipped to the top
- moved STDBY 48.5 mm to (19.6, 5.03), flipped to the top
- moved R13 36.7 mm to (25.0, 5.12), turned to 270 degrees
- moved R12 33.5 mm to (17.4, 5.06), turned to 270 degrees
- moved C4 14.8 mm to (12.1, 46.2), turned to 90 degrees
- moved R14 9.87 mm to (13.6, 46.2), turned to 270 degrees
- moved R8 8.85 mm to (3.75, 37.4), turned to 270 degrees
- moved C3 7.43 mm to (11.9, 31.9), turned to 270 degrees
- moved C1 6.18 mm to (12.7, 45.5), turned to 180 degrees
- moved R0 5.40 mm to (17.6, 54.7)
- moved MUX 4.49 mm to (12.2, 35.3)
- moved TP4056 2.40 mm to (13.8, 40.2), turned to 270 degrees
- moved R15 2.23 mm to (20.2, 34.2), turned to 270 degrees
- moved C2 2.20 mm to (5.23, 10.1), turned to 270 degrees
- moved LED1 0.41 mm to (12.2, 10.1)
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Connections:
- new net VEE: MUX.7
- net GND: no longer MUX.7
- net TP_B+: now also TP4056.8
- net VCC: no longer TP4056.8
Routing:
- net CHRG: track 3.09 -> 44.4 mm
- net STDBY: track 2.63 -> 38.5 mm
- net MUX_X2: track 63.9 -> 42.2 mm
- net E_LEFT_B: track 6.81 -> 27.1 mm
- net MUX_X0: track 34.9 -> 53.7 mm
- net WS_OUT: track 55.3 -> 71.5 mm
- net VCC: track 408.5 -> 422.2 mm, vias 4 -> 6
- net N$8: track 15.1 -> 2.25 mm, vias 1 -> 0
- net MUX_X1: track 46.1 -> 33.9 mm
- net TP_B+: track 4.96 -> 16.3 mm, vias 0 -> 3
- net MUX_X7: track 30.9 -> 40.9 mm
- net N$5: track 11.4 -> 2.63 mm, vias 1 -> 0
- net B+: track 40.7 -> 32.5 mm, vias 1 -> 2
- net EM: track 227.9 -> 235.5 mm
- net EM_ENABLE: track 43.1 -> 50.7 mm, vias 1 -> 2
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Other:
- board text added: "2022.01"
- board text added: "GND VCC"
- board text removed: "+"
- board text removed: "-"

Commit message: Fix unmatching PCB board version 2.7 (issue #22)
Parts:
- moved CHRG 48.5 mm to (19.2, 53.5), flipped to the bottom
- moved STDBY 48.5 mm to (21.9, 53.5), flipped to the bottom
- moved R13 36.7 mm to (17.9, 41.1), turned to 0 degrees
- moved R12 33.5 mm to (17.9, 38.6), turned to 0 degrees
- moved C4 14.8 mm to (4.21, 33.7), turned to 0 degrees
- moved R14 9.87 mm to (5.90, 40.0), turned to 0 degrees
- moved R8 8.85 mm to (-4.42, 40.8), turned to 180 degrees
- moved C3 7.43 mm to (17.7, 36.5), turned to 0 degrees
- moved C1 6.18 mm to (7.40, 48.7), turned to 90 degrees
- moved R0 5.40 mm to (12.2, 54.7)
- moved MUX 4.49 mm to (12.2, 30.8)
- moved TP4056 2.40 mm to (11.6, 39.3), turned to 0 degrees
- moved R15 2.23 mm to (17.9, 34.5), turned to 180 degrees
- moved C2 2.20 mm to (7.05, 8.91), turned to 90 degrees
- moved LED1 0.41 mm to (12.2, 9.65)
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Connections:
- removed net VEE: MUX.7
- net GND: now also MUX.7
- net TP_B+: no longer TP4056.8
- net VCC: now also TP4056.8
Routing:
- net CHRG: track 44.4 -> 3.09 mm
- net STDBY: track 38.5 -> 2.63 mm
- net MUX_X2: track 42.2 -> 63.9 mm
- net E_LEFT_B: track 27.1 -> 6.81 mm
- net MUX_X0: track 53.7 -> 34.9 mm
- net WS_OUT: track 71.5 -> 55.3 mm
- net VCC: track 422.2 -> 408.5 mm, vias 6 -> 4
- net N$8: track 2.25 -> 15.1 mm, vias 0 -> 1
- net MUX_X1: track 33.9 -> 46.1 mm
- net TP_B+: track 16.3 -> 4.96 mm, vias 3 -> 0
- net MUX_X7: track 40.9 -> 30.9 mm
- net N$5: track 2.63 -> 11.4 mm, vias 0 -> 1
- net B+: track 32.5 -> 40.7 mm, vias 2 -> 1
- net EM: track 235.5 -> 227.9 mm
- net EM_ENABLE: track 50.7 -> 43.1 mm, vias 2 -> 1
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Other:
- board text added: "+"
- board text added: "-"
- board text added: "2023.10"
- board text removed: "2022.01"
- board text removed: "2022.10"
- board text removed: "GND VCC"
